Commit message: Add PSIM results, setup loco-mujoco on kbot, and restructure MuJoCo folder

File: MuJoCo/kbot/urdf/robot_legs.urdf (robot description, URDF)
Before this commit: robot converted_robot, 14 links, 13 joints
Links:
- link KD_D_102L_L_Hip_Yoke_Drive: geometry visual mesh filename=C:/96v_gan_humanoid_drive/MuJoCo/kbot/urdf/meshes/KD_D_102L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
- link KD_D_102R: geometry visual mesh filename=C:/96v_gan_humanoid_drive/MuJoCo/kbot/urdf/meshes/KD_D_102R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
- link KD_D_301L_L_Femur_Lower_Drive: geometry visual mesh filename=C:/96v_gan_humanoid_drive/MuJoCo/kbot/urdf/meshes/KD_D_301L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
- link KD_D_301R: geometry visual mesh filename=C:/96v_gan_humanoid_drive/MuJoCo/kbot/urdf/meshes/KD_D_301R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
- link KD_D_401L_L_Shin_Drive: geometry visual mesh filename=C:/96v_gan_humanoid_drive/MuJoCo/kbot/urdf/meshes/KD_D_401L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
- link KD_D_401R: geometry visual mesh filename=C:/96v_gan_humanoid_drive/MuJoCo/kbot/urdf/meshes/KD_D_401R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
- link LFootBushing_GPF_1517_12: geometry visual mesh filename=C:/96v_gan_humanoid_drive/MuJoCo/kbot/urdf/meshes/LFootBush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
- link L_Hip_Roll_RS03: geometry visual mesh filename=C:/96v_gan_humanoid_drive/MuJoCo/kbot/urdf/meshes/L_Hip_Rol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
- link L_Hip_Roll_RS03_2: geometry visual mesh filename=C:/96v_gan_humanoid_drive/MuJoCo/kbot/urdf/meshes/L_Hip_Rol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
- link RFootBushing_GPF_1517_12: geometry visual mesh filename=C:/96v_gan_humanoid_drive/MuJoCo/kbot/urdf/meshes/RFootBush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

File: phase1/matlab/urdf/robot_legs.urdf (robot description, URDF)
Before this commit: robot converted_robot, 14 links, 13 joints
Links:
- link KD_D_102L_L_Hip_Yoke_Drive: geometry visual mesh filename=C:/96v_gan_humanoid_drive/MuJoCo/kbot/urdf/meshes/KD_D_102L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
- link KD_D_102R: geometry visual mesh filename=C:/96v_gan_humanoid_drive/MuJoCo/kbot/urdf/meshes/KD_D_102R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
- link KD_D_301L_L_Femur_Lower_Drive: geometry visual mesh filename=C:/96v_gan_humanoid_drive/MuJoCo/kbot/urdf/meshes/KD_D_301L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
- link KD_D_301R: geometry visual mesh filename=C:/96v_gan_humanoid_drive/MuJoCo/kbot/urdf/meshes/KD_D_301R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
- link KD_D_401L_L_Shin_Drive: geometry visual mesh filename=C:/96v_gan_humanoid_drive/MuJoCo/kbot/urdf/meshes/KD_D_401L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
- link KD_D_401R: geometry visual mesh filename=C:/96v_gan_humanoid_drive/MuJoCo/kbot/urdf/meshes/KD_D_401R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
- link LFootBushing_GPF_1517_12: geometry visual mesh filename=C:/96v_gan_humanoid_drive/MuJoCo/kbot/urdf/meshes/LFootBush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
- link L_Hip_Roll_RS03: geometry visual mesh filename=C:/96v_gan_humanoid_drive/MuJoCo/kbot/urdf/meshes/L_Hip_Rol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
- link L_Hip_Roll_RS03_2: geometry visual mesh filename=C:/96v_gan_humanoid_drive/MuJoCo/kbot/urdf/meshes/L_Hip_Rol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
- link RFootBushing_GPF_1517_12: geometry visual mesh filename=C:/96v_gan_humanoid_drive/MuJoCo/kbot/urdf/meshes/RFootBush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
